Commit message: fixed cohan_sim for ROS2 and some working launch files

File: src/cohan2.0_navigation/cohan_sim_navigation/robots/pr2.urdf (robot description, URDF)
Before this commit: robot pr2, 95 links, 94 joints
Links:
- link base_link: geometry collision mesh filename=package://cohan_sim_navigation/robots/meshes/base_v0/base_L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; visual mesh filename=package://cohan_sim_navigation/robots/meshes/base_v0/base.d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
- link bl_caster_l_wheel_link: geometry collision cylinder length=0.034 radius=0.074792; visual mesh filename=package://cohan_sim_navigation/robots/meshes/base_v0/wheel.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
- link bl_caster_r_wheel_link: geometry collision cylinder length=0.034 radius=0.074792; visual mesh filename=package://cohan_sim_navigation/robots/meshes/base_v0/wheel.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
- link bl_caster_rotation_link: geometry collision mesh filename=package://cohan_sim_navigation/robots/meshes/base_v0/caster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; visual mesh filename=package://cohan_sim_navigation/robots/meshes/base_v0/caster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
- link br_caster_l_wheel_link: geometry collision cylinder length=0.034 radius=0.074792; visual mesh filename=package://cohan_sim_navigation/robots/meshes/base_v0/wheel.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
- link br_caster_r_wheel_link: geometry collision cylinder length=0.034 radius=0.074792; visual mesh filename=package://cohan_sim_navigation/robots/meshes/base_v0/wheel.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
- link br_caster_rotation_link: geometry collision mesh filename=package://cohan_sim_navigation/robots/meshes/base_v0/caster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; visual mesh filename=package://cohan_sim_navigation/robots/meshes/base_v0/caster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
- link fl_caster_l_wheel_link: geometry collision cylinder length=0.034 radius=0.074792; visual mesh filename=package://cohan_sim_navigation/robots/meshes/base_v0/wheel.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
- link fl_caster_r_wheel_link: geometry collision cylinder length=0.034 radius=0.074792; visual mesh filename=package://cohan_sim_navigation/robots/meshes/base_v0/wheel.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
- link fl_caster_rotation_link: geometry collision mesh filename=package://cohan_sim_navigation/robots/meshes/base_v0/caster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; visual mesh filename=package://cohan_sim_navigation/robots/meshes/base_v0/caster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
- link fr_caster_l_wheel_link: geometry collision cylinder length=0.034 radius=0.074792; visual mesh filename=package://cohan_sim_navigation/robots/meshes/base_v0/wheel.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
- link fr_caster_r_wheel_link: geometry collision cylinder length=0.034 radius=0.074792; visual mesh filename=package://cohan_sim_navigation/robots/meshes/base_v0/wheel.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
- link fr_caster_rotation_link: geometry collision mesh filename=package://cohan_sim_navigation/robots/meshes/base_v0/caster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; visual mesh filename=package://cohan_sim_navigation/robots/meshes/base_v0/caster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
- link head_mount_link: geometry collision sphere radius=0.0005; visual mesh filename=package://cohan_sim_navigation/robots/meshes/sensors/kinect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 scale=0.001 0.001 0.001
- link head_pan_link: geometry collision mesh filename=package://cohan_sim_navigation/robots/meshes/head_v0/head_p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; visual mesh filename=package://cohan_sim_navigation/robots/meshes/head_v0/head_p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
- link head_tilt_link: geometry collision mesh filename=package://cohan_sim_navigation/robots/meshes/head_v0/head_t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; visual mesh filename=package://cohan_sim_navigation/robots/meshes/head_v0/head_t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
- link l_elbow_flex_link: geometry collision mesh filename=package://cohan_sim_navigation/robots/meshes/upper_arm_v0/e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; visual mesh filename=package://cohan_sim_navigation/robots/meshes/upper_arm_v0/e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
- link l_forearm_link: geometry collision mesh filename=package://cohan_sim_navigation/robots/meshes/forearm_v0/for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; visual mesh filename=package://cohan_sim_navigation/robots/meshes/forearm_v0/for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
- link l_forearm_roll_link: geometry collision mesh filename=package://cohan_sim_navigation/robots/meshes/upper_arm_v0/f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; visual mesh filename=package://cohan_sim_navigation/robots/meshes/upper_arm_v0/f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
- link l_gripper_l_finger_link: geometry collision mesh filename=package://cohan_sim_navigation/robots/meshes/gripper_v0/l_f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; visual mesh filename=package://cohan_sim_navigation/robots/meshes/gripper_v0/l_f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
- link l_gripper_l_finger_tip_link: geometry collision mesh filename=package://cohan_sim_navigation/robots/meshes/gripper_v0/l_f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; visual mesh filename=package://cohan_sim_navigation/robots/meshes/gripper_v0/l_f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
- link l_gripper_palm_link: geometry collision mesh filename=package://cohan_sim_navigation/robots/meshes/gripper_v0/gri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; visual mesh filename=package://cohan_sim_navigation/robots/meshes/gripper_v0/gri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
- link l_gripper_r_finger_link: geometry collision mesh filename=package://cohan_sim_navigation/robots/meshes/gripper_v0/l_f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; visual mesh filename=package://cohan_sim_navigation/robots/meshes/gripper_v0/l_f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
- link l_gripper_r_finger_tip_link: geometry collision mesh filename=package://cohan_sim_navigation/robots/meshes/gripper_v0/l_f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; visual mesh filename=package://cohan_sim_navigation/robots/meshes/gripper_v0/l_f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
- link l_shoulder_lift_link: geometry collision mesh filename=package://cohan_sim_navigation/robots/meshes/shoulder_v0/sh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; visual mesh filename=package://cohan_sim_navigation/robots/meshes/shoulder_v0/sh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
- link l_shoulder_pan_link: geometry collision mesh filename=package://cohan_sim_navigation/robots/meshes/shoulder_v0/sh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; visual mesh filename=package://cohan_sim_navigation/robots/meshes/shoulder_v0/sh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
- link l_upper_arm_link: geometry collision mesh filename=package://cohan_sim_navigation/robots/meshes/upper_arm_v0/u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; visual mesh filename=package://cohan_sim_navigation/robots/meshes/upper_arm_v0/u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
- link l_upper_arm_roll_link: geometry collision mesh filename=package://cohan_sim_navigation/robots/meshes/shoulder_v0/up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; visual mesh filename=package://cohan_sim_navigation/robots/meshes/shoulder_v0/up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
- link l_wrist_flex_link: geometry collision mesh filename=package://cohan_sim_navigation/robots/meshes/forearm_v0/wri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; visual mesh filename=package://cohan_sim_navigation/robots/meshes/forearm_v0/wri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
- link l_wrist_roll_link: geometry collision mesh filename=package://cohan_sim_navigation/robots/meshes/forearm_v0/wri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; visual mesh filename=package://cohan_sim_navigation/robots/meshes/forearm_v0/wri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
- link laser_tilt_mount_link: geometry collision mesh filename=package://cohan_sim_navigation/robots/meshes/tilting_laser_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; visual mesh filename=package://cohan_sim_navigation/robots/meshes/tilting_laser_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
- link r_elbow_flex_link: geometry collision mesh filename=package://cohan_sim_navigation/robots/meshes/upper_arm_v0/e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; visual mesh filename=package://cohan_sim_navigation/robots/meshes/upper_arm_v0/e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
- link r_forearm_link: geometry collision mesh filename=package://cohan_sim_navigation/robots/meshes/forearm_v0/for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; visual mesh filename=package://cohan_sim_navigation/robots/meshes/forearm_v0/for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
- link r_forearm_roll_link: geometry collision mesh filename=package://cohan_sim_navigation/robots/meshes/upper_arm_v0/f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; visual mesh filename=package://cohan_sim_navigation/robots/meshes/upper_arm_v0/f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
- link r_gripper_l_finger_link: geometry collision mesh filename=package://cohan_sim_navigation/robots/meshes/gripper_v0/l_f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; visual mesh filename=package://cohan_sim_navigation/robots/meshes/gripper_v0/l_f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
- link r_gripper_l_finger_tip_link: geometry collision mesh filename=package://cohan_sim_navigation/robots/meshes/gripper_v0/l_f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; visual mesh filename=package://cohan_sim_navigation/robots/meshes/gripper_v0/l_f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
- link r_gripper_palm_link: geometry collision mesh filename=package://cohan_sim_navigation/robots/meshes/gripper_v0/gri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; visual mesh filename=package://cohan_sim_navigation/robots/meshes/gripper_v0/gri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
- link r_gripper_r_finger_link: geometry collision mesh filename=package://cohan_sim_navigation/robots/meshes/gripper_v0/l_f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; visual mesh filename=package://cohan_sim_navigation/robots/meshes/gripper_v0/l_f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
- link r_gripper_r_finger_tip_link: geometry collision mesh filename=package://cohan_sim_navigation/robots/meshes/gripper_v0/l_f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; visual mesh filename=package://cohan_sim_navigation/robots/meshes/gripper_v0/l_f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
- link r_shoulder_lift_link: geometry collision mesh filename=package://cohan_sim_navigation/robots/meshes/shoulder_v0/sh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; visual mesh filename=package://cohan_sim_navigation/robots/meshes/shoulder_v0/sh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
- link r_shoulder_pan_link: geometry collision mesh filename=package://cohan_sim_navigation/robots/meshes/shoulder_v0/sh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; visual mesh filename=package://cohan_sim_navigation/robots/meshes/shoulder_v0/sh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
- link r_upper_arm_link: geometry collision mesh filename=package://cohan_sim_navigation/robots/meshes/upper_arm_v0/u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; visual mesh filename=package://cohan_sim_navigation/robots/meshes/upper_arm_v0/u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
- link r_upper_arm_roll_link: geometry collision mesh filename=package://cohan_sim_navigation/robots/meshes/shoulder_v0/up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; visual mesh filename=package://cohan_sim_navigation/robots/meshes/shoulder_v0/up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
- link r_wrist_flex_link: geometry collision mesh filename=package://cohan_sim_navigation/robots/meshes/forearm_v0/wri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; visual mesh filename=package://cohan_sim_navigation/robots/meshes/forearm_v0/wri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
- link r_wrist_roll_link: geometry collision mesh filename=package://cohan_sim_navigation/robots/meshes/forearm_v0/wri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; visual mesh filename=package://cohan_sim_navigation/robots/meshes/forearm_v0/wri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
- link torso_lift_link: geometry collision mesh filename=package://cohan_sim_navigation/robots/meshes/torso_v0/torso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; visual mesh filename=package://cohan_sim_navigation/robots/meshes/torso_v0/torso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
